File: PCB/I2C_connectors.sch (KiCad schematic (older format))
At the start: 10 parts, among them J10 3-way_power_jumper, J11 3-way_power_jumper, J4 Conn_01x04_Male, J5 Conn_01x04_Male, J8 Conn_01x04_Male, J9 Conn_01x04_Male

Commit message: Fixing all the paths
Parts:
- J10, J11: footprint ARCL:3-way_power_jumper -> other:3-way_power_jumper; symbol ARCL:3-way_power_jumper -> other:3-way_power_jumper
Changed lines of the file:
@@
 $EndComp
 $Comp
-L ARCL:3-way_power_jumper J?
+L other:3-way_power_jumper J?
 U 1 1 5FD48E56
 P 5650 4300
@@
 F 0 "J11" V 5654 4488 50  0000 L CNN
 F 1 "3-way_power_jumper" V 5745 4488 50  0000 L CNN
-F 2 "ARCL:3-way_power_jumper" H 5650 4050 50  0001 C CNN
+F 2 "other:3-way_power_jumper" H 5650 4050 50  0001 C CNN
 F 3 "" H 5650 4300 50  0001 C CNN
 	1    5650 4300
@@
 $EndComp
 $Comp
-L ARCL:3-way_power_jumper J?
+L other:3-way_power_jumper J?
 U 1 1 5FD48E5C
 P 5650 1900
@@
 F 0 "J10" V 5654 2088 50  0000 L CNN
 F 1 "3-way_power_jumper" V 5745 2088 50  0000 L CNN
-F 2 "ARCL:3-way_power_jumper" H 5650 1650 50  0001 C CNN
+F 2 "other:3-way_power_jumper" H 5650 1650 50  0001 C CNN
 F 3 "" H 5650 1900 50  0001 C CNN
 	1    5650 1900
