File: PCB/SPI_connectors.sch (KiCad schematic (older format))
At the start: 6 parts, among them J18 Conn_01x06_Male, J19 Conn_01x06_Male, J20 Conn_01x06_Male, J21 Conn_01x06_Male, J22 3-way_power_jumper, J23 3-way_power_jumper

Commit message: Fixing all the paths
Parts:
- J22, J23: footprint ARCL:3-way_power_jumper -> other:3-way_power_jumper; symbol ARCL:3-way_power_jumper -> other:3-way_power_jumper
Changed lines of the file:
@@
 $EndComp
 $Comp
-L ARCL:3-way_power_jumper J?
+L other:3-way_power_jumper J?
 U 1 1 5FD9007E
 P 6100 3950
 AR Path="/5FD33A77/5FD9007E" Ref="J?"  Part="1"
 AR Path="/5FD55215/5FD9007E" Ref="J23"  Part="1"
+AR Path="/5FD9007E" Ref="J23"  Part="1"
 F 0 "J23" V 6104 4138 50  0000 L CNN
 F 1 "3-way_power_jumper" V 6195 4138 50  0000 L CNN
-F 2 "ARCL:3-way_power_jumper" H 6100 3700 50  0001 C CNN
+F 2 "other:3-way_power_jumper" H 6100 3700 50  0001 C CNN
 F 3 "" H 6100 3950 50  0001 C CNN
 	1    6100 3950
@@
 $EndComp
 $Comp
-L ARCL:3-way_power_jumper J?
+L other:3-way_power_jumper J?
 U 1 1 5FD90AC7
 P 6100 1450
 AR Path="/5FD33A77/5FD90AC7" Ref="J?"  Part="1"
 AR Path="/5FD55215/5FD90AC7" Ref="J22"  Part="1"
+AR Path="/5FD90AC7" Ref="J22"  Part="1"
 F 0 "J22" V 6104 1638 50  0000 L CNN
 F 1 "3-way_power_jumper" V 6195 1638 50  0000 L CNN
-F 2 "ARCL:3-way_power_jumper" H 6100 1200 50  0001 C CNN
+F 2 "other:3-way_power_jumper" H 6100 1200 50  0001 C CNN
 F 3 "" H 6100 1450 50  0001 C CNN
 	1    6100 1450
