File: PCB/teensy_breakout.sch (KiCad schematic (older format))
At the start: 29 parts, among them J1 Conn_01x02_Male, J2 Conn_01x03_Male, J24 Conn_01x03_Male, J25 Conn_01x03_Male, J29 Conn_01x03_Male, J3 Conn_01x03_Male, J30 Conn_01x03_Male, J6 Conn_01x03_Male, J7 Conn_01x02_Male, U1 Teensy4.0, U2 Pololu_D24V22Fx

Commit message: Fixing all the paths
Parts:
- U2: footprint ARCL:Pololu_D24V22Fx_THT -> pololu:Pololu_D24V22Fx_THT; symbol ARCL:Pololu_D24V22Fx -> pololu:Pololu_D24V22Fx
Changed lines of the file:
@@
 $EndComp
 $Comp
-L ARCL:Pololu_D24V22Fx U2
+L pololu:Pololu_D24V22Fx U2
 U 1 1 5FD008AD
 P 8700 4600
 F 0 "U2" H 8725 5020 50  0000 C CNN
 F 1 "Pololu_D24V22Fx" H 8725 4929 50  0000 C CNN
-F 2 "ARCL:Pololu_D24V22Fx_THT" H 8700 4200 50  0001 C CNN
+F 2 "pololu:Pololu_D24V22Fx_THT" H 8700 4200 50  0001 C CNN
 F 3 "" H 8700 4200 50  0001 C CNN
 	1    8700 4600
